File: Diseño_Circuitos/Arduino/Bluetooth_Module.sch (KiCad schematic (older format))
At the start: 7 parts

Commit message: schematic completed
Parts:
- gave numbers to parts that had none: 7
Changed lines of the file:
@@
 LIBS:FT232RL
 LIBS:HC-05
+LIBS:L293DD
 LIBS:arduino-cache
 EELAYER 25 0
@@
 $Descr A4 11693 8268
 encoding utf-8
-Sheet 3 3
+Sheet 3 4
 Title ""
 Date ""
@@
 $EndDescr
 $Comp
-L HC-05 U?
+L HC-05 U4
 U 1 1 5F75322D
 P 5450 3400
-F 0 "U?" H 4850 4625 50  0000 L BNN
+F 0 "U4" H 4850 4625 50  0000 L BNN
 F 1 "HC-05" H 4850 2200 50  0000 L BNN
 F 2 "XCVR_HC-05" H 5450 3400 50  0001 L BNN
@@
 $EndComp
 $Comp
-L Conn_01x02 J?
+L Conn_01x02 J8
 U 1 1 5F753234
 P 3950 2000
-F 0 "J?" H 3950 2100 50  0000 C CNN
+F 0 "J8" H 3950 2100 50  0000 C CNN
 F 1 "Conn_01x02" H 3950 1800 50  0000 C CNN
 F 2 "" H 3950 2000 50  0001 C CNN
@@
 $EndComp
 $Comp
-L +3.3V #PWR?
+L +3.3V #PWR063
 U 1 1 5F75323B
 P 3650 1900
-F 0 "#PWR?" H 3650 1750 50  0001 C CNN
+F 0 "#PWR063" H 3650 1750 50  0001 C CNN
 F 1 "+3.3V" H 3650 2040 50  0000 C CNN
 F 2 "" H 3650 1900 50  0001 C CNN
@@
 $EndComp
 $Comp
-L +3.3VP #PWR?
+L +3.3VP #PWR064
 U 1 1 5F753241
 P 3650 2250
-F 0 "#PWR?" H 3800 2200 50  0001 C CNN
+F 0 "#PWR064" H 3800 2200 50  0001 C CNN
 F 1 "+3.3VP" H 3650 2350 50  0000 C CNN
 F 2 "" H 3650 2250 50  0001 C CNN
@@
 $EndComp
 $Comp
-L +3.3VP #PWR?
+L +3.3VP #PWR065
 U 1 1 5F753247
 P 6850 2250
-F 0 "#PWR?" H 7000 2200 50  0001 C CNN
+F 0 "#PWR065" H 7000 2200 50  0001 C CNN
 F 1 "+3.3VP" H 6850 2350 50  0000 C CNN
 F 2 "" H 6850 2250 50  0001 C CNN
@@
 $EndComp
 $Comp
-L C_Small C?
+L C_Small C17
 U 1 1 5F75324D
 P 6850 2450
-F 0 "C?" H 6860 2520 50  0000 L CNN
+F 0 "C17" H 6860 2520 50  0000 L CNN
 F 1 "100nF" H 6860 2370 50  0000 L CNN
 F 2 "" H 6850 2450 50  0000 C CNN
@@
 $EndComp
 $Comp
-L GND #PWR?
+L GND #PWR066
 U 1 1 5F753254
 P 6850 2650
-F 0 "#PWR?" H 6850 2400 50  0001 C CNN
+F 0 "#PWR066" H 6850 2400 50  0001 C CNN
 F 1 "GND" H 6850 2500 50  0000 C CNN
 F 2 "" H 6850 2650 50  0001 C CNN
@@
 NoConn ~ 6250 3800
 $Comp
-L +3.3VP #PWR?
+L +3.3VP #PWR067
 U 1 1 5F753263
 P 6350 2200
-F 0 "#PWR?" H 6500 2150 50  0001 C CNN
+F 0 "#PWR067" H 6500 2150 50  0001 C CNN
 F 1 "+3.3VP" H 6350 2300 50  0000 C CNN
 F 2 "" H 6350 2200 50  0001 C CNN
@@
 $EndComp
 $Comp
-L GND #PWR?
+L GND #PWR068
 U 1 1 5F753269
 P 6300 4450
-F 0 "#PWR?" H 6300 4200 50  0001 C CNN
+F 0 "#PWR068" H 6300 4200 50  0001 C CNN
 F 1 "GND" H 6300 4300 50  0000 C CNN
 F 2 "" H 6300 4450 50  0001 C CNN
@@
 $EndComp
 $Comp
-L SW_Push SW?
+L SW_Push SW6
 U 1 1 5F75326F
 P 6700 3600
-F 0 "SW?" H 6750 3700 50  0000 L CNN
+F 0 "SW6" H 6750 3700 50  0000 L CNN
 F 1 "SW_Push" H 6700 3540 50  0000 C CNN
 F 2 "" H 6700 3800 50  0001 C CNN
@@
 $EndComp
 $Comp
-L +3.3VP #PWR?
+L +3.3VP #PWR069
 U 1 1 5F753276
 P 7150 3600
-F 0 "#PWR?" H 7300 3550 50  0001 C CNN
+F 0 "#PWR069" H 7300 3550 50  0001 C CNN
 F 1 "+3.3VP" V 7200 3650 50  0000 C CNN
 F 2 "" H 7150 3600 50  0001 C CNN
@@
 $EndComp
 $Comp
-L R_Small R?
+L R_Small R24
 U 1 1 5F75327C
 P 6400 3800
-F 0 "R?" H 6430 3820 50  0000 L CNN
+F 0 "R24" H 6430 3820 50  0000 L CNN
 F 1 "10k" H 6430 3760 50  0000 L CNN
 F 2 "" H 6400 3800 50  0000 C CNN
@@
 $EndComp
 $Comp
-L GND #PWR?
+L GND #PWR070
 U 1 1 5F753283
 P 6400 4000
-F 0 "#PWR?" H 6400 3750 50  0001 C CNN
+F 0 "#PWR070" H 6400 3750 50  0001 C CNN
 F 1 "GND" H 6400 3850 50  0000 C CNN
 F 2 "" H 6400 4000 50  0001 C CNN
@@
 NoConn ~ 6250 3500
 $Comp
-L R_Small R?
+L R_Small R23
 U 1 1 5F75328A
 P 6900 3300
-F 0 "R?" H 6930 3320 50  0000 L CNN
+F 0 "R23" H 6930 3320 50  0000 L CNN
 F 1 "2k" H 6930 3260 50  0000 L CNN
 F 2 "" H 6900 3300 50  0000 C CNN
@@
 $EndComp
 $Comp
-L LED_ALT D?
+L LED_ALT D13
 U 1 1 5F753291
 P 7250 3300
-F 0 "D?" H 7250 3400 50  0000 C CNN
+F 0 "D13" H 7250 3400 50  0000 C CNN
 F 1 "LED_ALT" H 7250 3200 50  0000 C CNN
 F 2 "" H 7250 3300 50  0000 C CNN
@@
 $EndComp
 $Comp
-L GND #PWR?
+L GND #PWR071
 U 1 1 5F753298
 P 7500 3300
-F 0 "#PWR?" H 7500 3050 50  0001 C CNN
+F 0 "#PWR071" H 7500 3050 50  0001 C CNN
 F 1 "GND" H 7500 3150 50  0000 C CNN
 F 2 "" H 7500 3300 50  0001 C CNN
@@
 Wire Wire Line
 	4500 2900 4650 2900
+$Comp
+L +3.3VP #PWR072
+U 1 1 5F762086
+P 7750 2250
+F 0 "#PWR072" H 7900 2200 50  0001 C CNN
+F 1 "+3.3VP" H 7750 2350 50  0000 C CNN
+F 2 "" H 7750 2250 50  0001 C CNN
+F 3 "" H 7750 2250 50  0001 C CNN
+	1    7750 2250
+	1    0    0    -1
+$EndComp
+$Comp
+L PWR_FLAG #FLG073
+U 1 1 5F7620A1
+P 7750 2550
+F 0 "#FLG073" H 7750 2625 50  0001 C CNN
+F 1 "PWR_FLAG" H 7750 2700 50  0000 C CNN
+F 2 "" H 7750 2550 50  0001 C CNN
+F 3 "" H 7750 2550 50  0001 C CNN
+	1    7750 2550
+	-1   0    0    1
+$EndComp
+Wire Wire Line
+	7750 2250 7750 2550
 $EndSCHEMATC

Commit message: pcb components placed
Parts:
- C17: footprint (none) -> custom footprints:C_0805_HandSoldering
- D13: footprint (none) -> custom footprints:LED_0805
- J8: footprint (none) -> custom footprints:Pin_Header_Straight_1x02_Pitch2.54mm
- R23, R24: footprint (none) -> custom footprints:R_0805_HandSoldering
- SW6: footprint (none) -> custom footprints:SW_SPST_FSMSM
- U4: footprint XCVR_HC-05 -> custom footprints:XCVR_HC-05
Changed lines of the file:
@@
 F 0 "U4" H 4850 4625 50  0000 L BNN
 F 1 "HC-05" H 4850 2200 50  0000 L BNN
-F 2 "XCVR_HC-05" H 5450 3400 50  0001 L BNN
+F 2 "custom footprints:XCVR_HC-05" H 5450 3400 50  0001 L BNN
 F 3 "HuiCheng" H 5450 3400 50  0001 L BNN
 F 4 "v1.0" H 5450 3400 50  0001 L BNN "Campo4"
@@
 F 0 "J8" H 3950 2100 50  0000 C CNN
 F 1 "Conn_01x02" H 3950 1800 50  0000 C CNN
-F 2 "" H 3950 2000 50  0001 C CNN
+F 2 "custom footprints:Pin_Header_Straight_1x02_Pitch2.54mm" H 3950 2000 50  0001 C CNN
 F 3 "" H 3950 2000 50  0001 C CNN
 	1    3950 2000
@@
 F 0 "C17" H 6860 2520 50  0000 L CNN
 F 1 "100nF" H 6860 2370 50  0000 L CNN
-F 2 "" H 6850 2450 50  0000 C CNN
+F 2 "custom footprints:C_0805_HandSoldering" H 6850 2450 50  0001 C CNN
 F 3 "" H 6850 2450 50  0000 C CNN
 	1    6850 2450
@@
 F 0 "SW6" H 6750 3700 50  0000 L CNN
 F 1 "SW_Push" H 6700 3540 50  0000 C CNN
-F 2 "" H 6700 3800 50  0001 C CNN
+F 2 "custom footprints:SW_SPST_FSMSM" H 6700 3800 50  0001 C CNN
 F 3 "" H 6700 3800 50  0001 C CNN
 	1    6700 3600
@@
 F 0 "R24" H 6430 3820 50  0000 L CNN
 F 1 "10k" H 6430 3760 50  0000 L CNN
-F 2 "" H 6400 3800 50  0000 C CNN
+F 2 "custom footprints:R_0805_HandSoldering" H 6400 3800 50  0001 C CNN
 F 3 "" H 6400 3800 50  0000 C CNN
 	1    6400 3800
@@
 F 0 "R23" H 6930 3320 50  0000 L CNN
 F 1 "2k" H 6930 3260 50  0000 L CNN
-F 2 "" H 6900 3300 50  0000 C CNN
+F 2 "custom footprints:R_0805_HandSoldering" H 6900 3300 50  0001 C CNN
 F 3 "" H 6900 3300 50  0000 C CNN
 	1    6900 3300
@@
 F 0 "D13" H 7250 3400 50  0000 C CNN
 F 1 "LED_ALT" H 7250 3200 50  0000 C CNN
-F 2 "" H 7250 3300 50  0000 C CNN
+F 2 "custom footprints:LED_0805" H 7250 3300 50  0001 C CNN
 F 3 "" H 7250 3300 50  0000 C CNN
 	1    7250 3300
